Commit message: model_Update

File: newton/examples/ai_worker/ai_worker.urdf (robot description, URDF)
Before this commit: robot ffw_sg2_follower, 42 links, 41 joints
Links:
- link arm_base_link: geometry collision mesh filename=./ffw_description/meshes/common/follower/body_arm_assy.stl scale=0.001 0.001 0.001; visual mesh filename=./ffw_description/meshes/common/follower/body_arm_assy.stl scale=0.001 0.001 0.001
- link arm_l_link1: geometry collision mesh filename=./ffw_description/meshes/common/follower/arm_l_link1.stl scale=0.001 0.001 0.001; visual mesh filename=./ffw_description/meshes/common/follower/arm_l_link1.stl scale=0.001 0.001 0.001
- link arm_l_link2: geometry collision mesh filename=./ffw_description/meshes/common/follower/arm_l_link2.stl scale=0.001 0.001 0.001; visual mesh filename=./ffw_description/meshes/common/follower/arm_l_link2.stl scale=0.001 0.001 0.001
- link arm_l_link3: geometry collision mesh filename=./ffw_description/meshes/common/follower/arm_l_link3.stl scale=0.001 0.001 0.001; visual mesh filename=./ffw_description/meshes/common/follower/arm_l_link3.stl scale=0.001 0.001 0.001
- link arm_l_link4: geometry collision mesh filename=./ffw_description/meshes/common/follower/arm_l_link4.stl scale=0.001 0.001 0.001; visual mesh filename=./ffw_description/meshes/common/follower/arm_l_link4.stl scale=0.001 0.001 0.001
- link arm_l_link5: geometry collision mesh filename=./ffw_description/meshes/common/follower/arm_l_link5.stl scale=0.001 0.001 0.001; visual mesh filename=./ffw_description/meshes/common/follower/arm_l_link5.stl scale=0.001 0.001 0.001
- link arm_l_link6: geometry collision mesh filename=./ffw_description/meshes/common/follower/arm_l_link6.stl scale=0.001 0.001 0.001; visual mesh filename=./ffw_description/meshes/common/follower/arm_l_link6.stl scale=0.001 0.001 0.001
- link arm_l_link7: geometry collision mesh filename=./ffw_description/meshes/common/follower/arm_l_link7.stl scale=0.001 0.001 0.001; visual mesh filename=./ffw_description/meshes/common/follower/arm_l_link7.stl scale=0.001 0.001 0.001
- link arm_r_link1: geometry collision mesh filename=./ffw_description/meshes/common/follower/arm_r_link1.stl scale=0.001 0.001 0.001; visual mesh filename=./ffw_description/meshes/common/follower/arm_r_link1.stl scale=0.001 0.001 0.001
- link arm_r_link2: geometry collision mesh filename=./ffw_description/meshes/common/follower/arm_r_link2.stl scale=0.001 0.001 0.001; visual mesh filename=./ffw_description/meshes/common/follower/arm_r_link2.stl scale=0.001 0.001 0.001
- link arm_r_link3: geometry collision mesh filename=./ffw_description/meshes/common/follower/arm_r_link3.stl scale=0.001 0.001 0.001; visual mesh filename=./ffw_description/meshes/common/follower/arm_r_link3.stl scale=0.001 0.001 0.001
- link arm_r_link4: geometry collision mesh filename=./ffw_description/meshes/common/follower/arm_r_link4.stl scale=0.001 0.001 0.001; visual mesh filename=./ffw_description/meshes/common/follower/arm_r_link4.stl scale=0.001 0.001 0.001
- link arm_r_link5: geometry collision mesh filename=./ffw_description/meshes/common/follower/arm_r_link5.stl scale=0.001 0.001 0.001; visual mesh filename=./ffw_description/meshes/common/follower/arm_r_link5.stl scale=0.001 0.001 0.001
- link arm_r_link6: geometry collision mesh filename=./ffw_description/meshes/common/follower/arm_r_link6.stl scale=0.001 0.001 0.001; visual mesh filename=./ffw_description/meshes/common/follower/arm_r_link6.stl scale=0.001 0.001 0.001
- link arm_r_link7: geometry collision mesh filename=./ffw_description/meshes/common/follower/arm_r_link7.stl scale=0.001 0.001 0.001; visual mesh filename=./ffw_description/meshes/common/follower/arm_r_link7.stl scale=0.001 0.001 0.001
- link base_link: geometry collision mesh filename=./ffw_description/meshes/ffw_sg2_rev1_follower/base_mobile_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 scale=0.001 0.001 0.001; visual mesh filename=./ffw_description/meshes/ffw_sg2_rev1_follower/base_mobile_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 scale=0.001 0.001 0.001
- link camera_l_link: geometry collision box size=0.023 0.042 0.042; visual mesh filename=./ffw_description/meshes/common/follower/zedm.stl scale=0.001 0.001 0.001
- link camera_r_link: geometry collision box size=0.023 0.042 0.042; visual mesh filename=./ffw_description/meshes/common/follower/zedm.stl scale=0.001 0.001 0.001
- link gripper_l_rh_p12_rn_base: geometry collision mesh filename=./ffw_description/meshes/common/rh_p12_rn_a/base.stl scale=0.001 0.001 0.001; visual mesh filename=./ffw_description/meshes/common/rh_p12_rn_a/base.stl scale=0.001 0.001 0.001
- link gripper_l_rh_p12_rn_l1: geometry collision mesh filename=./ffw_description/meshes/common/rh_p12_rn_a/l1.stl scale=0.001 0.001 0.001; visual mesh filename=./ffw_description/meshes/common/rh_p12_rn_a/l1.stl scale=0.001 0.001 0.001
- link gripper_l_rh_p12_rn_l2: geometry collision mesh filename=./ffw_description/meshes/common/rh_p12_rn_a/l2.stl scale=0.001 0.001 0.001; visual mesh filename=./ffw_description/meshes/common/rh_p12_rn_a/l2.stl scale=0.001 0.001 0.001
- link gripper_l_rh_p12_rn_r1: geometry collision mesh filename=./ffw_description/meshes/common/rh_p12_rn_a/r1.stl scale=0.001 0.001 0.001; visual mesh filename=./ffw_description/meshes/common/rh_p12_rn_a/r1.stl scale=0.001 0.001 0.001
- link gripper_l_rh_p12_rn_r2: geometry collision mesh filename=./ffw_description/meshes/common/rh_p12_rn_a/r2.stl scale=0.001 0.001 0.001; visual mesh filename=./ffw_description/meshes/common/rh_p12_rn_a/r2.stl scale=0.001 0.001 0.001
- link gripper_r_rh_p12_rn_base: geometry collision mesh filename=./ffw_description/meshes/common/rh_p12_rn_a/base.stl scale=0.001 0.001 0.001; visual mesh filename=./ffw_description/meshes/common/rh_p12_rn_a/base.stl scale=0.001 0.001 0.001
- link gripper_r_rh_p12_rn_l1: geometry collision mesh filename=./ffw_description/meshes/common/rh_p12_rn_a/l1.stl scale=0.001 0.001 0.001; visual mesh filename=./ffw_description/meshes/common/rh_p12_rn_a/l1.stl scale=0.001 0.001 0.001
- link gripper_r_rh_p12_rn_l2: geometry collision mesh filename=./ffw_description/meshes/common/rh_p12_rn_a/l2.stl scale=0.001 0.001 0.001; visual mesh filename=./ffw_description/meshes/common/rh_p12_rn_a/l2.stl scale=0.001 0.001 0.001
- link gripper_r_rh_p12_rn_r1: geometry collision mesh filename=./ffw_description/meshes/common/rh_p12_rn_a/r1.stl scale=0.001 0.001 0.001; visual mesh filename=./ffw_description/meshes/common/rh_p12_rn_a/r1.stl scale=0.001 0.001 0.001
- link gripper_r_rh_p12_rn_r2: geometry collision mesh filename=./ffw_description/meshes/common/rh_p12_rn_a/r2.stl scale=0.001 0.001 0.001; visual mesh filename=./ffw_description/meshes/common/rh_p12_rn_a/r2.stl scale=0.001 0.001 0.001
- link head_link1: geometry collision mesh filename=./ffw_description/meshes/common/follower/head_link1.stl scale=0.001 0.001 0.001; visual mesh filename=./ffw_description/meshes/common/follower/head_link1.stl scale=0.001 0.001 0.001
- link head_link2: geometry collision mesh filename=./ffw_description/meshes/common/follower/head_link2.stl scale=0.001 0.001 0.001; visual mesh filename=./ffw_description/meshes/common/follower/head_link2.stl scale=0.001 0.001 0.001
- link left_wheel_drive_link: geometry collision mesh filename=./ffw_description/meshes/ffw_sg2_rev1_follower/left_wheel_d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 scale=0.001 0.001 0.001; visual mesh filename=./ffw_description/meshes/ffw_sg2_rev1_follower/left_wheel_d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 scale=0.001 0.001 0.001
- link left_wheel_steer_link: geometry collision mesh filename=./ffw_description/meshes/ffw_sg2_rev1_follower/left_wheel_s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 scale=0.001 0.001 0.001; visual mesh filename=./ffw_description/meshes/ffw_sg2_rev1_follower/left_wheel_s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 scale=0.001 0.001 0.001
- link lift_link: geometry collision mesh filename=./ffw_description/meshes/ffw_sg2_rev1_follower/lift_link.stl scale=0.001 0.001 0.001; visual mesh filename=./ffw_description/meshes/ffw_sg2_rev1_follower/lift_link.stl scale=0.001 0.001 0.001
- link rear_wheel_drive_link: geometry collision mesh filename=./ffw_description/meshes/ffw_sg2_rev1_follower/rear_wheel_d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 scale=0.001 0.001 0.001; visual mesh filename=./ffw_description/meshes/ffw_sg2_rev1_follower/rear_wheel_d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 scale=0.001 0.001 0.001
- link rear_wheel_steer_link: geometry collision mesh filename=./ffw_description/meshes/ffw_sg2_rev1_follower/rear_wheel_s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 scale=0.001 0.001 0.001; visual mesh filename=./ffw_description/meshes/ffw_sg2_rev1_follower/rear_wheel_s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 scale=0.001 0.001 0.001
- link right_wheel_drive_link: geometry collision mesh filename=./ffw_description/meshes/ffw_sg2_rev1_follower/right_wheel_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 scale=0.001 0.001 0.001; visual mesh filename=./ffw_description/meshes/ffw_sg2_rev1_follower/right_wheel_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 scale=0.001 0.001 0.001
- link right_wheel_steer_link: geometry collision mesh filename=./ffw_description/meshes/ffw_sg2_rev1_follower/right_wheel_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 scale=0.001 0.001 0.001; visual mesh filename=./ffw_description/meshes/ffw_sg2_rev1_follower/right_wheel_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 scale=0.001 0.001 0.001
